Commit message: change color of tower and create an own material file in our repo

File: raw_common/raw_description/urdf/tower/cam3d_tower.urdf.xacro (robot description, xacro)
@@ -20,5 +20,5 @@
           <box size="${depth} ${width} ${height}"/>
         </geometry>
-        <material name="DarkGrey" />
+        <material name="LightGrey" />
       </visual>
       <collision>

File: raw_robots/raw_hardware_config/youbot_hbrs2/urdf/youbot_hbrs2.urdf.xacro (robot description, xacro)
@@ -20,4 +20,5 @@
   <!-- materials for visualization -->
   <include filename="$(find youbot_description)/urdf/materials.urdf.xacro" />
+  <include filename="$(find raw_description)/urdf/materials.urdf.xacro" />
   <!-- additional sensors and other stuff -->
   <include filename="$(find raw_description)/urdf/tower/cam3d_tower.urdf.xacro" />

Commit message: uggly fix of calibration. Will be changed soon through Marcs Kinect model

File: raw_common/raw_description/urdf/tower/cam3d_tower.urdf.xacro (robot description, xacro)
@@ -5,5 +5,5 @@
        xmlns:xacro="http://ros.org/wiki/xacro">
   <include filename="$(find raw_description)/urdf/sensors/kinect.urdf.xacro" />
-  <property name="height" value="0.52" />
+  <property name="height" value="0.515" />
   <property name="width" value="0.03" />
   <property name="depth" value="0.03" />
@@ -37,5 +37,5 @@
   <!-- 3D camera on tower -->
   <xacro:kinect name="openni" parent="tower_link" ros_topic="/camera/rgb/points" tilt="0.61">
-    <origin xyz="0 0 ${height}" rpy="0 0 0" />
+    <origin xyz="0 -0.04 ${height-0.05}" rpy="0 0 0" />
   </xacro:kinect>
 </root>
