Commit message: add base laser scanner to our specific youbot file

File: raw_robots/raw_hardware_config/youbot_hbrs2/urdf/youbot_hbrs2.urdf.xacro (robot description, xacro)
@@ -20,8 +20,4 @@
   <!-- materials for visualization -->
   <include filename="$(find youbot_description)/urdf/materials.urdf.xacro" />
-  <include filename="$(find raw_description)/urdf/materials.urdf.xacro" />
-  <!-- additional sensors and other stuff -->
-  <include filename="$(find raw_description)/urdf/tower/cam3d_tower.urdf.xacro" />
-  <!--include filename="$(find youbot_description)/urdf/sensors/asus_xtion.urdf.xacro" />-->
   <!-- Now we can start using the macros included above to define the actual youbot -->
   <!-- The first use of a macro.  This one was defined in base.urdf.xacro above.
@@ -43,5 +39,13 @@
     <origin xyz="0 0 0" rpy="0 0 0" />
   </xacro:youbot_gripper>
-  <!-- 3D camera on tower -->
+  <!-- BRSU SPECIFIC STUFF -->
+  <include filename="$(find raw_description)/urdf/materials.urdf.xacro" />
+  <include filename="$(find raw_description)/urdf/tower/cam3d_tower.urdf.xacro" />
+  <!--include filename="$(find youbot_description)/urdf/sensors/asus_xtion.urdf.xacro" />-->
+  <!-- base laser rear -->
+  <xacro:hokuyo_urg04_laser name="base_laser_rear" parent="base" ros_topic="scan_rear" update_rate="10" min_angle="-1.57" max_angle="1.57" >
+     <origin xyz="-0.3 0 -0.03" rpy="0 0 ${M_PI}" />
+  </xacro:hokuyo_urg04_laser>
+  <!-- tower with 3D camera -->
   <xacro:cam3d_tower name="tower" parent="plate_link">
     <origin xyz="-0.05 0 0.025" rpy="0 0 0" />

Commit message: adjust tower position

File: raw_robots/raw_hardware_config/youbot_hbrs2/urdf/youbot_hbrs2.urdf.xacro (robot description, xacro)
@@ -49,5 +49,5 @@
   <!-- tower with 3D camera -->
   <xacro:cam3d_tower name="tower" parent="plate_link">
-    <origin xyz="-0.05 0 0.025" rpy="0 0 0" />
+    <origin xyz="-0.025 0 0.025" rpy="0 0 0" />
   </xacro:cam3d_tower>
   <!-- ASUS Xtion on arm joint 4
