Commit message: Fix wrong size of simulated arena

File: raw_environments/raw_gazebo_worlds/common/worlds/brsu-home.urdf (robot description, URDF)
Before this commit: robot arena, 12 links, 11 joints
Links:
- link wall_1: geometry collision box size=4.04 0.015 0.3; visual box size=4.04 0.015 0.3
- link wall_3: geometry collision box size=4.04 0.015 0.3; visual box size=4.04 0.015 0.3
Joints:
- joint join1: origin xyz=2.2 0 0 rpy=0 0 0 -> xyz=2.02 0 0 rpy=0 0 0
- joint join2: origin xyz=-2.2 -1.215 0 rpy=0 0 0 -> xyz=-2.02 -1.215 0 rpy=0 0 0
- joint join5: origin xyz=-2.2 -0.4 0 rpy=0 0 0 -> xyz=-2.02 -0.4 0 rpy=0 0 0
- joint join6: origin xyz=-2.2 0 0 rpy=0 0 0 -> xyz=-2.02 0 0 rpy=0 0 0

Commit message: Fix wrong size of simulated area (urdf file)

File: raw_environments/raw_gazebo_worlds/common/worlds/brsu-home.urdf (robot description, URDF)
Before this commit: robot arena, 12 links, 11 joints
Links:
- link wall_10: geometry collision box size=0.5 2.44 0.11; visual box size=0.5 2.44 0.11
- link wall_2: geometry collision box size=0.015 -2.44 0.3; visual box size=0.015 -2.44 0.3
Joints:
- joint join2: origin xyz=-2.02 -1.215 0 rpy=0 0 0 -> xyz=-2.02 -1.22 0 rpy=0 0 0
