Commit message: fix kinect frame_ids so that is working in simulation

File: raw_common/raw_description/urdf/sensors/kinect.gazebo.xacro (robot description, xacro)
@@ -22,5 +22,5 @@
         <pointCloudTopicName>/camera/depth/points</pointCloudTopicName>
         <cameraInfoTopicName>/camera/camera_info</cameraInfoTopicName>
-        <frameName>/openni_camera_depth_optical_frame</frameName>
+        <frameName>/openni_depth_optical_frame</frameName>
         <distortion_k1>0.000000001</distortion_k1>
         <distortion_k2>0.000000001</distortion_k2>

File: raw_common/raw_description/urdf/sensors/kinect.urdf.xacro (robot description, xacro)
@@ -33,7 +33,7 @@
     <origin xyz="0 0.018 0" rpy="0 0 0" />
     <parent link="${name}_camera" />
-    <child link="${name}_camera_depth_frame" />
+    <child link="${name}_depth_frame" />
   </joint>
-  <link name="${name}_camera_depth_frame">
+  <link name="${name}_depth_frame">
     <inertial>
       <mass value="0.01" />
@@ -46,8 +46,8 @@
   <joint name="${name}_camera_depth_optical_joint" type="fixed">
     <origin xyz="0 0 0" rpy="${-M_PI/2} 0 ${-M_PI/2}" />
-    <parent link="${name}_camera_depth_frame" />
-    <child link="${name}_camera_depth_optical_frame" />
+    <parent link="${name}_depth_frame" />
+    <child link="${name}_depth_optical_frame" />
   </joint>
-  <link name="${name}_camera_depth_optical_frame">
+  <link name="${name}_depth_optical_frame">
     <inertial>
       <mass value="0.001" />
@@ -61,7 +61,7 @@
     <origin xyz="0 -0.005 0" rpy="0 0 0" />
     <parent link="${name}_camera" />
-    <child link="${name}_camera_rgb_frame" />
+    <child link="${name}_rgb_frame" />
   </joint>
-  <link name="${name}_camera_rgb_frame">
+  <link name="${name}_rgb_frame">
     <inertial>
       <mass value="0.001" />
@@ -74,8 +74,8 @@
   <joint name="${name}_camera_rgb_optical_joint" type="fixed">
     <origin xyz="0 0 0" rpy="${-M_PI/2} 0 ${-M_PI/2}" />
-    <parent link="${name}_camera_rgb_frame" />
-    <child link="${name}_camera_rgb_optical_frame" />
+    <parent link="${name}_rgb_frame" />
+    <child link="${name}_rgb_optical_frame" />
   </joint>
-  <link name="${name}_camera_rgb_optical_frame">
+  <link name="${name}_rgb_optical_frame">
     <inertial>
       <mass value="0.001" />
