Commit message: add aluminium profiles

File: raw_environments/raw_gazebo_objects/common/objects/alu_profil_f20_black.urdf.xacro (robot description, xacro)
@@ -1,32 +1,5 @@
 <?xml version="1.0"?>
-<robot name="objects" 	xmlns:xacro="http://ros.org/wiki/xacro">
-	<include filename="$(find raw_description)/urdf/materials.urdf.xacro" />
-	<xacro:macro name="rectangle" params="name parent width height length color *origin">
-		<link name="${name}_link">
-			<inertial>
-				<insert_block name="origin" />
-				<mass value="10.0" />
-			    <inertia  ixx="1.0" ixy="0.0"  ixz="0.0"  iyy="1.0"  iyz="0.0"  izz="1.0" />
-			</inertial>
-			<visual>
-				<insert_block name="origin" />
-				<geometry>
-					<box size="${length} ${width} ${height}"/>
-				</geometry>
-			</visual>
-			<collision>
-				<insert_block name="origin" />
-				<geometry>
-			   		<box size="${length} ${width} ${height}"/>
-				</geometry>
-			</collision >
-		</link>
-		<gazebo reference="${name}_link">
-			<material>${color}</material>
-			<selfCollide>true</selfCollide>
-		</gazebo>
-	</xacro:macro>
-	<xacro:rectangle name="square1" parent="dummy_link" width="0.05" height="0.05" length="0.05" color="Gazebo/Black">
-	    <origin xyz="0 0 0.25" rpy="0 0 0" />
-	</xacro:rectangle>
+<robot name="alu_profil_f20_black" xmlns:xacro="http://ros.org/wiki/xacro">
+	<include filename="$(find raw_gazebo_objects)/common/templates/box.urdf.xacro" />
+	<xacro:box_template name="alu_profil_f20_black" length="0.1" width="0.02" height="0.02" color="Gazebo/Black" />
 </robot>
