Commit message: add correct weight of objects

File: raw_environments/raw_gazebo_objects/common/objects/adapter_sleeve_r20.urdf.xacro (robot description, xacro)
@@ -2,4 +2,4 @@
 <robot name="adapter_sleeve_r20" xmlns:xacro="http://ros.org/wiki/xacro">
 	<include filename="$(find raw_gazebo_objects)/common//templates/model.urdf.xacro" />
-	<xacro:model_template name="adapter_sleeve_r20" model_filename="adapter_sleeve_r20.dae" scale="0.001" height="0.045"/>
+	<xacro:model_template name="adapter_sleeve_r20" model_filename="adapter_sleeve_r20.dae" scale="0.001" height="0.045" weight="0.010"/>
 </robot>

File: raw_environments/raw_gazebo_objects/common/objects/adapter_sleeve_v20.urdf.xacro (robot description, xacro)
@@ -2,4 +2,4 @@
 <robot name="adapter_sleeve_v20" xmlns:xacro="http://ros.org/wiki/xacro">
 	<include filename="$(find raw_gazebo_objects)/common//templates/model.urdf.xacro" />
-	<xacro:model_template name="adapter_sleeve_v20" model_filename="adapter_sleeve_v20.dae" scale="0.001" height="0.045"/>
+	<xacro:model_template name="adapter_sleeve_v20" model_filename="adapter_sleeve_v20.dae" scale="0.001" height="0.045"  weight="0.015"/>
 </robot>

File: raw_environments/raw_gazebo_objects/common/objects/aluprofil_f20_100_gray.urdf.xacro (robot description, xacro)
@@ -2,4 +2,4 @@
 <robot name="aluprofil_f20_100_gray" xmlns:xacro="http://ros.org/wiki/xacro">
 	<include filename="$(find raw_gazebo_objects)/common/templates/model.urdf.xacro" />
-	<xacro:model_template name="aluprofil_f20_100_gray" model_filename="aluprofil_f20_100_gray.dae" scale="0.001"  height="0.1"/>
+	<xacro:model_template name="aluprofil_f20_100_gray" model_filename="aluprofil_f20_100_gray.dae" scale="0.001"  height="0.1"  weight="0.05"/>
 </robot>

File: raw_environments/raw_gazebo_objects/common/objects/aluprofil_s40_100_gray.urdf.xacro (robot description, xacro)
@@ -2,4 +2,4 @@
 <robot name="aluprofil_s40_100_gray" xmlns:xacro="http://ros.org/wiki/xacro">
 	<include filename="$(find raw_gazebo_objects)/common/templates/model.urdf.xacro" />
-	<xacro:model_template name="aluprofil_s40_100_gray" model_filename="aluprofil_s40_100_gray.dae" scale="0.001"  height="0.1"/>
+	<xacro:model_template name="aluprofil_s40_100_gray" model_filename="aluprofil_s40_100_gray.dae" scale="0.001"  height="0.1"  weight="0.185"/>
 </robot>

File: raw_environments/raw_gazebo_objects/common/objects/bolt_m20_100.urdf.xacro (robot description, xacro)
@@ -2,4 +2,4 @@
 <robot name="bolt_m20_100" xmlns:xacro="http://ros.org/wiki/xacro">
 	<include filename="$(find raw_gazebo_objects)/common/templates/model.urdf.xacro" />
-	<xacro:model_template name="bolt_m20_100" model_filename="bolt_m20_100.dae" scale="0.001"  height="0.01"/>
+	<xacro:model_template name="bolt_m20_100" model_filename="bolt_m20_100.dae" scale="0.001"  height="0.01"  weight="0.290"/>
 </robot>

File: raw_environments/raw_gazebo_objects/common/objects/bolt_m20_180.urdf.xacro (robot description, xacro)
@@ -2,4 +2,4 @@
 <robot name="bolt_m20_180" xmlns:xacro="http://ros.org/wiki/xacro">
 	<include filename="$(find raw_gazebo_objects)/common/templates/model.urdf.xacro" />
-	<xacro:model_template name="bolt_m20_180" model_filename="bolt_m20_180.dae" scale="0.001"  height="0.01"/>
+	<xacro:model_template name="bolt_m20_180" model_filename="bolt_m20_180.dae" scale="0.001"  height="0.01"  weight="0.477"/>
 </robot>

File: raw_environments/raw_gazebo_objects/common/objects/nut_m20.urdf.xacro (robot description, xacro)
@@ -2,4 +2,4 @@
 <robot name="nut_m20" xmlns:xacro="http://ros.org/wiki/xacro">
 	<include filename="$(find raw_gazebo_objects)/common/templates/model.urdf.xacro" />
-	<xacro:model_template name="nut_m20" model_filename="nut_m20.dae" scale="0.001"  height="0.01"/>
+	<xacro:model_template name="nut_m20" model_filename="nut_m20.dae" scale="0.001"  height="0.01"  weight="0.068"/>
 </robot>

File: raw_environments/raw_gazebo_objects/common/objects/nut_m30.urdf.xacro (robot description, xacro)
@@ -2,4 +2,4 @@
 <robot name="nut_m30" xmlns:xacro="http://ros.org/wiki/xacro">
 	<include filename="$(find raw_gazebo_objects)/common/templates/model.urdf.xacro" />
-	<xacro:model_template name="nut_m30" model_filename="nut_m30.dae" scale="0.001"  height="0.01"/>
+	<xacro:model_template name="nut_m30" model_filename="nut_m30.dae" scale="0.001"  height="0.01"  weight="0.215"/>
 </robot>

File: raw_environments/raw_gazebo_objects/common/templates/model.urdf.xacro (robot description, xacro)
@@ -14,9 +14,9 @@
 	    xmlns:physics="http://playerstage.sourceforge.net/gazebo/xmlschema/#physics"
 	    xmlns:xacro="http://www.ros.org/wiki/xacro">
-	<xacro:macro name="model_template" params="name model_filename scale height">
+	<xacro:macro name="model_template" params="name model_filename scale height weight">
 		<link name="${name}_link">
 			<inertial>
 				<origin xyz="0 0 ${-height / 2}" rpy="0 0 0" />
-				<mass value="0.001" />
+				<mass value="${weight}" />
 			    <inertia  ixx="1.0" ixy="0.0"  ixz="0.0"  iyy="1.0"  iyz="0.0"  izz="1.0" />
 			</inertial>
