Commit message: add additional @work objects to simulation

File: raw_environments/raw_gazebo_objects/common/templates/box.urdf.xacro (robot description, xacro)
@@ -1,14 +1,13 @@
 <?xml version="1.0"?>
 <robot name="box_template" xmlns:xacro="http://ros.org/wiki/xacro">
-	<include filename="$(find raw_description)/urdf/materials.urdf.xacro" />
 	<xacro:macro name="box_template" params="name length width height color">
 		<link name="${name}_link">
 			<inertial>
-				<origin xyz="${length / 2} ${width / 2} ${height / 2}" rpy="0 0 0" />
+				<origin xyz="${length / 32} ${width / 32} ${height / 32}" rpy="0 0 0" />
 				<mass value="10.0" />
 			    <inertia  ixx="1.0" ixy="0.0"  ixz="0.0"  iyy="1.0"  iyz="0.0"  izz="1.0" />
 			</inertial>
 			<visual>
-				<origin xyz="${length / 2} ${width / 2} ${height / 2}" rpy="0 0 0" />
+				<origin xyz="${length / 32} ${width / 32} ${height / 32}" rpy="0 0 0" />
 				<geometry>
 					<box size="${length} ${width} ${height}" />
@@ -16,5 +15,5 @@
 			</visual>
 			<collision>
-				<origin xyz="${length / 2} ${width / 2} ${height / 2}" rpy="0 0 0" />
+				<origin xyz="${length / 32} ${width / 32} ${height / 32}" rpy="0 0 0" />
 				<geometry>
 			   		<box size="${length} ${width} ${height}" />

Commit message: add friction and reduce mass

File: raw_environments/raw_gazebo_objects/common/templates/box.urdf.xacro (robot description, xacro)
@@ -5,5 +5,5 @@
 			<inertial>
 				<origin xyz="${length / 32} ${width / 32} ${height / 32}" rpy="0 0 0" />
-				<mass value="10.0" />
+				<mass value="0.001" />
 			    <inertia  ixx="1.0" ixy="0.0"  ixz="0.0"  iyy="1.0"  iyz="0.0"  izz="1.0" />
 			</inertial>
@@ -22,4 +22,8 @@
 		</link>
 		<gazebo reference="${name}_link">
+			<mu1 value="100.0" />
+		    <mu2 value="100.0" />
+            <kp  value="1000000.0" />
+            <kd  value="1.0" />
 			<material>${color}</material>
 			<selfCollide>true</selfCollide>

File: raw_environments/raw_gazebo_objects/common/templates/model.urdf.xacro (robot description, xacro)
@@ -18,5 +18,5 @@
 			<inertial>
 				<origin xyz="0 0 ${-height / 2}" rpy="0 0 0" />
-				<mass value="10.0" />
+				<mass value="0.001" />
 			    <inertia  ixx="1.0" ixy="0.0"  ixz="0.0"  iyy="1.0"  iyz="0.0"  izz="1.0" />
 			</inertial>
@@ -35,4 +35,8 @@
 		</link>
 		<gazebo reference="${name}_link">
+		    <mu1 value="100.0" />
+		    <mu2 value="100.0" />
+            <kp  value="1000000.0" />
+            <kd  value="1.0" />
 			<selfCollide>true</selfCollide>
 		</gazebo>

File: raw_environments/raw_gazebo_objects/common/templates/nut.urdf.xacro (robot description, xacro)
@@ -5,5 +5,5 @@
 			<inertial>
 				<origin xyz="${radius / 32} ${radius / 32} ${height / 32}" rpy="0 0 0" />
-				<mass value="10.0" />
+				<mass value="0.001" />
 			    <inertia  ixx="1.0" ixy="0.0"  ixz="0.0"  iyy="1.0"  iyz="0.0"  izz="1.0" />
 			</inertial>
@@ -22,4 +22,8 @@
 		</link>
 		<gazebo reference="${name}_link">
+			<mu1 value="100.0" />
+		    <mu2 value="100.0" />
+            <kp  value="1000000.0" />
+            <kd  value="1.0" />
 			<material>${color}</material>
 			<selfCollide>true</selfCollide>

File: raw_environments/raw_gazebo_objects/common/templates/pipe.urdf.xacro (robot description, xacro)
@@ -5,5 +5,5 @@
 			<inertial>
 				<origin xyz="${radius / 32} ${radius / 32} ${height / 32}" rpy="0 0 0" />
-				<mass value="10.0" />
+				<mass value="0.001" />
 			    <inertia  ixx="1.0" ixy="0.0"  ixz="0.0"  iyy="1.0"  iyz="0.0"  izz="1.0" />
 			</inertial>
@@ -22,4 +22,8 @@
 		</link>
 		<gazebo reference="${name}_link">
+			<mu1 value="100.0" />
+		    <mu2 value="100.0" />
+            <kp  value="1000000.0" />
+            <kd  value="1.0" />
 			<material>${color}</material>
 			<selfCollide>true</selfCollide>
